Commit message: tested launch cmu urdf

File: interbotix_ros_xslocobots/interbotix_xslocobot_descriptions/urdf/cmu_locobot/cmu_locobot_description.urdf (robot description, URDF)
Before this commit: robot locobot, 25 links, 24 joints
Links:
- link ar_tag: geometry collision mesh filename=package://interbotix_xslocobot_descriptions/meshes/cmu_loco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; visual mesh filename=package://interbotix_xslocobot_descriptions/meshes/cmu_loco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
- link arm_base_link: geometry collision mesh filename=package://interbotix_xslocobot_descriptions/meshes/cmu_loco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; visual mesh filename=package://interbotix_xslocobot_descriptions/meshes/cmu_loco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
- link base_link: geometry collision cylinder length=0.10938 radius=0.178; visual mesh filename=package://interbotix_xslocobot_descriptions/meshes/cmu_loco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
- link cam_mount: geometry collision mesh filename=package://interbotix_xslocobot_descriptions/meshes/cmu_loco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; visual mesh filename=package://interbotix_xslocobot_descriptions/meshes/cmu_loco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
- link camera_link: geometry collision mesh filename=package://interbotix_xslocobot_descriptions/meshes/cmu_loco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; visual mesh filename=package://interbotix_xslocobot_descriptions/meshes/cmu_loco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
- link elbow_link: geometry collision mesh filename=package://interbotix_xslocobot_descriptions/meshes/cmu_loco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; visual mesh filename=package://interbotix_xslocobot_descriptions/meshes/cmu_loco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
- link finger_l: geometry collision mesh filename=package://interbotix_xslocobot_descriptions/meshes/cmu_loco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; visual mesh filename=package://interbotix_xslocobot_descriptions/meshes/cmu_loco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
- link finger_r: geometry collision mesh filename=package://interbotix_xslocobot_descriptions/meshes/cmu_loco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; visual mesh filename=package://interbotix_xslocobot_descriptions/meshes/cmu_loco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
- link forearm_link: geometry collision mesh filename=package://interbotix_xslocobot_descriptions/meshes/cmu_loco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; visual mesh filename=package://interbotix_xslocobot_descriptions/meshes/cmu_loco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
- link gripper_link: geometry collision mesh filename=package://interbotix_xslocobot_descriptions/meshes/cmu_loco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; visual mesh filename=package://interbotix_xslocobot_descriptions/meshes/cmu_loco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
- link head_pan_link: geometry collision mesh filename=package://interbotix_xslocobot_descriptions/meshes/cmu_loco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; visual mesh filename=package://interbotix_xslocobot_descriptions/meshes/cmu_loco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
- link head_tilt_link: geometry collision mesh filename=package://interbotix_xslocobot_descriptions/meshes/cmu_loco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; visual mesh filename=package://interbotix_xslocobot_descriptions/meshes/cmu_loco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
- link plate_1: geometry collision mesh filename=package://interbotix_xslocobot_descriptions/meshes/cmu_loco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; visual mesh filename=package://interbotix_xslocobot_descriptions/meshes/cmu_loco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
- link plate_2: geometry collision mesh filename=package://interbotix_xslocobot_descriptions/meshes/cmu_loco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; visual mesh filename=package://interbotix_xslocobot_descriptions/meshes/cmu_loco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
- link shoulder_link: geometry collision mesh filename=package://interbotix_xslocobot_descriptions/meshes/cmu_loco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; visual mesh filename=package://interbotix_xslocobot_descriptions/meshes/cmu_loco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
- link wheel_left_link: geometry collision cylinder length=0.0206 radius=0.0352; visual mesh filename=package://interbotix_xslocobot_descriptions/meshes/cmu_loco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
- link wheel_right_link: geometry collision cylinder length=0.0206 radius=0.0350; visual mesh filename=package://interbotix_xslocobot_descriptions/meshes/cmu_loco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
- link wrist_link: geometry collision mesh filename=package://interbotix_xslocobot_descriptions/meshes/cmu_loco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; visual mesh filename=package://interbotix_xslocobot_descriptions/meshes/cmu_loco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
