Commit message: modified urdf to launch locobotcmu, passed gazebo sim launch

File: interbotix_ros_xslocobots/interbotix_xslocobot_descriptions/urdf/arms/mobile_arm.urdf.xacro (robot description, xacro)
@@ -5,10 +5,15 @@
       <joint name="arm_base_link_joint" type="fixed">
         <axis xyz="0 0 0"/>
-        <xacro:if value="${arm_type == 'mobile_px100'}">
-          <origin rpy="0 0 0" xyz="0.111126 0 0.0095"/>
-        </xacro:if> <!-- arm_type == 'mobile_px100' -->
-        <xacro:if value="${arm_type != 'mobile_px100'}">
-          <origin rpy="0 0 0" xyz="0.097277 0 0.0095"/>
-        </xacro:if> <!-- arm_type != 'mobile_px100' -->
+        <xacro:if value="${robot_model_var.startswith('locobotcmu')}">
+          <origin rpy="0 0 0" xyz="0 0 0.001"/>
+        </xacro:if> <!-- robot_model_var.startswith('locobotcmu') -->
+        <xacro:unless value="${robot_model_var.startswith('locobotcmu')}">
+          <xacro:if value="${arm_type == 'mobile_px100'}">
+            <origin rpy="0 0 0" xyz="0.111126 0 0.0095"/>
+          </xacro:if> <!-- arm_type == 'mobile_px100' -->
+          <xacro:if value="${arm_type != 'mobile_px100'}">
+            <origin rpy="0 0 0" xyz="0.097277 0 0.0095"/>
+          </xacro:if> <!-- arm_type != 'mobile_px100' -->
+        </xacro:unless> <!-- not robot_model_var.startswith('locobotcmu') -->
         <parent link="${robot_name}/plate_link"/>
         <child link="${robot_name}/arm_base_link"/>

File: interbotix_ros_xslocobots/interbotix_xslocobot_descriptions/urdf/arms/mobile_wx200.urdf.xacro (robot description, xacro)
@@ -35,40 +35,66 @@
   <xacro:include filename="$(find interbotix_xslocobot_descriptions)/urdf/arms/arm_control.urdf.xacro"/>
   <xacro:include filename="$(find interbotix_xslocobot_descriptions)/urdf/arms/ar_tag.urdf.xacro"/>
-  <link name="${robot_name}/arm_base_link">
-    <visual>
-      <origin
-        rpy="${pi/2} 0 ${pi/2}"
-        xyz="-0.095773 0 -0.10565023"/>
-      <geometry>
-        <mesh
-          filename="${mesh_directory}/base.stl"
-          scale="0.001 0.001 0.001"/>
-      </geometry>
-      <material name="interbotix_black"/>
-    </visual>
-    <collision>
-      <origin
-        rpy="${pi/2} 0 ${pi/2}"
-        xyz="-0.095773 0 -0.10565023"/>
-      <geometry>
-        <mesh
-          filename="${mesh_directory}/base.stl"
-          scale="0.001 0.001 0.001"/>
-      </geometry>
-    </collision>
-    <inertial>
-      <origin
-        rpy="${pi/2} 0 ${pi/2}"
-        xyz="-0.0001350000 -0.0000266286 0.0338755000"/>
-      <mass value="0.379673"/>
-      <inertia
-        ixx="0.0004351000"
-        iyy="0.0004452000"
-        izz="0.0005731000"
-        ixy="0.0000000707"
-        ixz="0.0000000266"
-        iyz="-0.0000022881"/>
-    </inertial>
-  </link>
+  <xacro:if value="${robot_model_var.startswith('locobotcmu')}">
+    <link name="${robot_name}/arm_base_link">
+        <inertial>
+            <origin rpy="0 0 0" xyz="-1.86027246940057E-08 -1.84987775462994E-08 0.0400356424684456"/>
+            <mass value="0.531491686912019"/>
+            <inertia ixx="0.000533657400855491" ixy="-4.44205269454465E-09" ixz="2.11078566024265E-10" iyy="0.000533665698902565" iyz="5.02029005902419E-11" izz="0.00071572082392375"/>
+        </inertial>
+        <visual>
+            <origin rpy="0 0 0" xyz="0 0 0"/>
+            <geometry>
+                <mesh filename="package://interbotix_xslocobot_descriptions/meshes/cmu_locobot_meshes/arm_base_link.STL"/>
+            </geometry>
+            <material name="">
+                <color rgba="0.792156862745098 0.819607843137255 0.933333333333333 1"/>
+            </material>
+        </visual>
+        <collision>
+            <origin rpy="0 0 0" xyz="0 0 0"/>
+            <geometry>
+                <mesh filename="package://interbotix_xslocobot_descriptions/meshes/cmu_locobot_meshes/arm_base_link.STL"/>
+            </geometry>
+        </collision>
+    </link>
+  </xacro:if> <!-- robot_model.startswith('locobotcmu_wx200') -->
+  <xacro:unless value="${robot_model_var.startswith('locobotcmu')}">
+    <link name="${robot_name}/arm_base_link">
+      <visual>
+        <origin
+          rpy="${pi/2} 0 ${pi/2}"
+          xyz="-0.095773 0 -0.10565023"/>
+        <geometry>
+          <mesh
+            filename="${mesh_directory}/base.stl"
+            scale="0.001 0.001 0.001"/>
+        </geometry>
+        <material name="interbotix_black"/>
+      </visual>
+      <collision>
+        <origin
+          rpy="${pi/2} 0 ${pi/2}"
+          xyz="-0.095773 0 -0.10565023"/>
+        <geometry>
+          <mesh
+            filename="${mesh_directory}/base.stl"
+            scale="0.001 0.001 0.001"/>
+        </geometry>
+      </collision>
+      <inertial>
+        <origin
+          rpy="${pi/2} 0 ${pi/2}"
+          xyz="-0.0001350000 -0.0000266286 0.0338755000"/>
+        <mass value="0.379673"/>
+        <inertia
+          ixx="0.0004351000"
+          iyy="0.0004452000"
+          izz="0.0005731000"
+          ixy="0.0000000707"
+          ixz="0.0000000266"
+          iyz="-0.0000022881"/>
+      </inertial>
+    </link>
+  </xacro:unless> <!-- !robot_model.startswith('locobotcmu_wx200') -->
   <joint name="waist" type="revolute">
     <axis xyz="0 0 1"/>
@@ -78,7 +104,14 @@
       upper="${waist_limit_upper}"
       velocity="${waist_limit_vel}"/>
-    <origin
-      rpy="0 0 0"
-      xyz="0 0 0.066175"/>
+    <xacro:if value="${robot_model_var.startswith('locobotcmu')}">
+      <origin
+        rpy="0 0 0"
+        xyz="0 0 0.072"/>
+    </xacro:if> <!-- robot_model.startswith('locobotcmu_wx200') -->
+    <xacro:unless value="${robot_model_var.startswith('locobotcmu')}">
+      <origin
+        rpy="0 0 0"
+        xyz="0 0 0.066175"/>
+    </xacro:unless> <!-- !robot_model.startswith('locobotcmu_wx200') -->
     <parent
       link="${robot_name}/arm_base_link"/>

File: interbotix_ros_xslocobots/interbotix_xslocobot_descriptions/urdf/camera_tower.urdf.xacro (robot description, xacro)
@@ -40,3 +40,39 @@
     </gazebo>
   </xacro:macro>
+  <xacro:macro name="locobotcmu_camera_tower">
+    <joint name="camera_tower" type="fixed">
+        <origin rpy="0 0 0" xyz="-0.03751 0 0.1331"/>
+        <parent link="${robot_name}/base_link"/>
+        <child link="${robot_name}/camera_tower_link"/>
+        <axis xyz="0 0 0"/>
+    </joint>
+    <link name="${robot_name}/camera_tower_link">
+      <inertial>
+            <origin rpy="0 0 0" xyz="0.00357169217419921 -0.000144750803528887 0.178406861295468"/>
+            <mass value="0.508068698311304"/>
+            <inertia ixx="0.0159487749924762" ixy="9.45818767875249E-08" ixz="-0.000266253609478166" iyy="0.0137751425461872" iyz="2.26699147122113E-06" izz="0.00331206257835318"/>
+        </inertial>
+        <visual>
+            <origin rpy="0 0 0" xyz="0 0 0"/>
+            <geometry>
+                <mesh filename="package://interbotix_xslocobot_descriptions/meshes/cmu_locobot_meshes/cam_mount.STL"/>
+            </geometry>
+            <material name="">
+                <color rgba="0.792156862745098 0.819607843137255 0.933333333333333 1"/>
+            </material>
+        </visual>
+        <collision>
+            <origin rpy="0 0 0" xyz="0 0 0"/>
+            <geometry>
+                <mesh filename="package://interbotix_xslocobot_descriptions/meshes/cmu_locobot_meshes/cam_mount.STL"/>
+            </geometry>
+        </collision>
+    </link>
+    <gazebo reference="${robot_name}/camera_tower_link">
+      <material>Gazebo/DarkGrey</material>
+    </gazebo>
+    <gazebo reference="camera_tower">
+      <disableFixedJointLumping>true</disableFixedJointLumping>
+    </gazebo>
+  </xacro:macro>
 </robot>

File: interbotix_ros_xslocobots/interbotix_xslocobot_descriptions/urdf/locobot.urdf.xacro (robot description, xacro)
@@ -18,4 +18,5 @@
   <xacro:property name="urdf_loc"         value="$(arg external_urdf_loc)"/>
   <xacro:property name="pi_offset"        value="0.00001"/>
+  <xacro:property name="robot_model_var"  value="$(arg robot_model)"/>
   <xacro:if value="${urdf_loc != ''}">
     <xacro:include filename="${urdf_loc}"/>
@@ -45,232 +46,269 @@
   </xacro:if> <!-- create3 -->
   <!-- ********************************** Plate **********************************  -->
-  <xacro:if value="${base_type == 'kobuki'}">
-    <xacro:plate>
-      <origin
-        rpy="0 0 0"
-        xyz="0.0 0 0.08825"/>
-      <inertial>
+  <xacro:if value="${robot_model_var.startswith('locobotcmu')}">
+    <xacro:locobotcmu_plate/>
+  </xacro:if> <!-- robot_model.startswith('locobotcmu_wx200') -->
+  <xacro:unless value="${robot_model_var.startswith('locobotcmu')}">
+    <xacro:if value="${base_type == 'kobuki'}">
+      <xacro:plate>
         <origin
           rpy="0 0 0"
-          xyz="0.050816 0 0.00475"/>
-        <mass value="0.571995"/>
-        <inertia
-          ixx="0.003115"
-          ixy="0"
-          ixz="0"
-          iyy="0.001813"
-          iyz="0"
-          izz="0.004919"/>
-      </inertial>
-    </xacro:plate>
-  </xacro:if> <!-- base_type == 'kobuki' -->
-  <xacro:if value="${base_type == 'create3'}">
-    <xacro:plate>
-      <origin
-        rpy="0 0 0"
-        xyz="0 0 0.0934"/>
-      <inertial>
+          xyz="0.0 0 0.08825"/>
+        <inertial>
+          <origin
+            rpy="0 0 0"
+            xyz="0.050816 0 0.00475"/>
+          <mass value="0.571995"/>
+          <inertia
+            ixx="0.003115"
+            ixy="0"
+            ixz="0"
+            iyy="0.001813"
+            iyz="0"
+            izz="0.004919"/>
+        </inertial>
+      </xacro:plate>
+    </xacro:if> <!-- base_type == 'kobuki' -->
+    <xacro:if value="${base_type == 'create3'}">
+      <xacro:plate>
         <origin
           rpy="0 0 0"
-          xyz="-0.005869 0 4.67E-03"/>
-        <mass value="0.807674"/>
-        <inertia
-          ixx="5.27E-03"
-          ixy="0"
-          ixz="0"
-          iyy="3.27E-03"
-          iyz="0"
-          izz="8.54E-03"/>
-      </inertial>
-    </xacro:plate>
-  </xacro:if> <!-- base_type == 'create3' -->
+          xyz="0 0 0.0934"/>
+        <inertial>
+          <origin
+            rpy="0 0 0"
+            xyz="-0.005869 0 4.67E-03"/>
+          <mass value="0.807674"/>
+          <inertia
+            ixx="5.27E-03"
+            ixy="0"
+            ixz="0"
+            iyy="3.27E-03"
+            iyz="0"
+            izz="8.54E-03"/>
+        </inertial>
+      </xacro:plate>
+    </xacro:if> <!-- base_type == 'create3' -->
+  </xacro:unless> <!-- !robot_model_var.startswith('locobotcmu_wx200') -->
   <!-- ********************************** Arm ********************************** -->
-  <xacro:if value="${arm_type != 'mobile_base'}">
-    <xacro:include filename="$(find interbotix_xslocobot_descriptions)/urdf/arms/mobile_arm.urdf.xacro"/>
-    <xacro:mobile_arm/>
-    <xacro:if value="${arm_type == 'mobile_wx200'}">
-      <xacro:if value="${base_type == 'kobuki'}">
-        <xacro:arm_cradle>
-          <origin
-            rpy="0 0 0"
-            xyz="0.0215 0 0.1195"/>
-        </xacro:arm_cradle>
-      </xacro:if> <!-- base_type == 'kobuki' -->
-      <xacro:if value="${base_type == 'create3'}">
-        <xacro:arm_cradle>
-          <origin
-            rpy="0 0 0"
-            xyz="0.037943 0 0.139"/>
-        </xacro:arm_cradle>
-      </xacro:if> <!-- base_type == 'create3' -->
-    </xacro:if> <!-- arm_type == 'mobile_wx200' -->
-  </xacro:if> <!-- arm_type != 'mobile_base' -->
+  <xacro:if value="${robot_model_var.startswith('locobotcmu')}">
+    <xacro:if value="${arm_type != 'mobile_base'}">
+      <xacro:include filename="$(find interbotix_xslocobot_descriptions)/urdf/arms/mobile_arm.urdf.xacro"/>
+      <xacro:mobile_arm/>
+    </xacro:if> <!-- arm_type != 'mobile_base' -->
+  </xacro:if> <!-- robot_model.startswith('locobotcmu_wx200') -->
+  <xacro:unless value="${robot_model_var.startswith('locobotcmu')}">
+    <xacro:if value="${arm_type != 'mobile_base'}">
+      <xacro:include filename="$(find interbotix_xslocobot_descriptions)/urdf/arms/mobile_arm.urdf.xacro"/>
+      <xacro:mobile_arm/>
+      <xacro:if value="${arm_type == 'mobile_wx200'}">
+        <xacro:if value="${base_type == 'kobuki'}">
+          <xacro:arm_cradle>
+            <origin
+              rpy="0 0 0"
+              xyz="0.0215 0 0.1195"/>
+          </xacro:arm_cradle>
+        </xacro:if> <!-- base_type == 'kobuki' -->
+        <xacro:if value="${base_type == 'create3'}">
+          <xacro:arm_cradle>
+            <origin
+              rpy="0 0 0"
+              xyz="0.037943 0 0.139"/>
+          </xacro:arm_cradle>
+        </xacro:if> <!-- base_type == 'create3' -->
+      </xacro:if> <!-- arm_type == 'mobile_wx200' -->
+    </xacro:if> <!-- arm_type != 'mobile_base' -->
+  </xacro:unless> <!-- !robot_model.startswith('locobotcmu_wx200') -->
   <!-- ********************************** Battery **********************************  -->
-  <xacro:if value="${base_type == 'kobuki'}">
-    <xacro:battery>
-      <origin
-        rpy="0 0 0"
-        xyz="-0.007 0 0.0125"/>
-    </xacro:battery>
-  </xacro:if> <!-- base_type == 'kobuki' -->
-  <xacro:if value="${base_type == 'create3'}">
-    <xacro:battery>
-      <origin
-        rpy="0 0 0"
-        xyz="-0.0345 0 0.010763"/>
-    </xacro:battery>
-  </xacro:if> <!-- base_type == 'create3' -->
-  <!-- ********************************** Camera Tower **********************************  -->
-  <xacro:if value="${base_type == 'kobuki'}">
-    <xacro:if value="${camera_tower_size == 'large'}">
-      <xacro:camera_tower>
+  <xacro:if value="${robot_model_var.startswith('locobotcmu')}">
+    <!-- Currently no battery for CMU locobot -->
+    <!-- TODO: add battery in the future -->
+  </xacro:if> <!-- robot_model.startswith('locobotcmu_wx200') -->
+  <xacro:unless value="${robot_model_var.startswith('locobotcmu')}">
+    <xacro:if value="${base_type == 'kobuki'}">
+      <xacro:battery>
         <origin
           rpy="0 0 0"
-          xyz="-0.023997 -0.000044 0.08823"/>
-        <inertial>
-          <origin
-            rpy="0 0 0"
-            xyz="-0.0372211000 -0.0026114300 0.1744600000"/>
-          <mass value="2.366224"/>
-          <inertia
-            ixx="0.0628500000"
-            ixy="0.0002152000"
-            ixz="0.0065630000"
-            iyy="0.0546000000"
-            iyz="-0.0004738000"
-            izz="0.0179300000"/>
-        </inertial>
-      </xacro:camera_tower>
-    </xacro:if> <!-- base_type == 'kobuki' && camera_tower_size == 'large' -->
-    <xacro:if value="${camera_tower_size == 'small'}">
-      <xacro:camera_tower>
+          xyz="-0.007 0 0.0125"/>
+      </xacro:battery>
+    </xacro:if> <!-- base_type == 'kobuki' -->
+    <xacro:if value="${base_type == 'create3'}">
+      <xacro:battery>
         <origin
           rpy="0 0 0"
-          xyz="-0.023997 -0.000044 0.08823"/>
-        <inertial>
-          <origin
-            rpy="0 0 0"
-            xyz="-0.0357703000 -0.0027068600 0.1560470000"/>
-          <mass value="2.282808"/>
-          <inertia
-            ixx="0.0461600000"
-            ixy="0.0002062000"
-            ixz="0.0052560000"
-            iyy="0.0384200000"
-            iyz="-0.0003600000"
-            izz="0.0169600000"/>
-        </inertial>
-      </xacro:camera_tower>
-    </xacro:if> <!-- base_type == 'kobuki' && camera_tower_size == 'small' -->
-  </xacro:if> <!-- base_type == 'kobuki' -->
-  <xacro:if value="${base_type == 'create3'}">
-    <xacro:if value="${camera_tower_size == 'large'}">
-      <xacro:camera_tower>
-        <origin
-          rpy="0 0 0"
-          xyz="-0.048271 0 0.10087"/>
-        <inertial>
-          <origin
-            rpy="0 0 0"
-            xyz="-0.025958 -0.003319 0.205872"/>
-          <mass value="2.514064"/>
-          <inertia
-            ixx="7.61E-02"
-            ixy="1.47E-04"
-            ixz="7.04E-03"
-            iyy="6.71E-02"
-            iyz="-9.41E-04"
-            izz="1.95E-02"/>
-        </inertial>
-      </xacro:camera_tower>
-    </xacro:if> <!-- base_type == 'create3' && camera_tower_size == 'large' -->
-    <xacro:if value="${camera_tower_size == 'small'}">
-      <xacro:camera_tower>
-        <origin
-          rpy="0 0 0"
-          xyz="-0.048271 0 0.10087"/>
-        <inertial>
-          <origin
-            rpy="0 0 0"
-            xyz="-0.024689 -0.003432 0.185408"/>
-          <mass value="2.430647"/>
-          <inertia
-            ixx="5.63E-02"
-            ixy="1.37E-04"
-            ixz="5.75E-03"
-            iyy="4.78E-02"
-            iyz="-7.70E-04"
-            izz="1.86E-02"/>
-        </inertial>
-      </xacro:camera_tower>
-    </xacro:if> <!-- base_type == 'create3' && camera_tower_size == 'small' -->
-  </xacro:if> <!-- base_type == 'create3' -->
-  <!-- ********************************** Pan & Tilt **********************************  -->
-  <xacro:if value="${base_type == 'kobuki'}">
-    <xacro:if value="${camera_tower_size == 'large'}">
-      <xacro:pan_and_tilt>
-        <origin
-          rpy="0 0 0"
-          xyz="0.047228 0 0.44425"/>
-      </xacro:pan_and_tilt>
-    </xacro:if> <!-- base_type == 'kobuki' && camera_tower_size == 'large' -->
-    <xacro:if value="${camera_tower_size == 'small'}">
-      <xacro:pan_and_tilt>
-        <origin
-          rpy="0 0 0"
-          xyz="0.047228 0 0.38425"/>
-      </xacro:pan_and_tilt>
-    </xacro:if> <!-- base_type == 'kobuki' && camera_tower_size == 'small' -->
-  </xacro:if> <!-- base_type == 'kobuki' -->
-  <xacro:if value="${base_type == 'create3'}">
-    <xacro:if value="${camera_tower_size == 'large'}">
-      <xacro:pan_and_tilt>
-        <origin
-          rpy="0 0 0"
-          xyz="0.061228 0 0.462"/>
-      </xacro:pan_and_tilt>
-    </xacro:if> <!-- base_type == 'create3' && camera_tower_size == 'large' -->
-    <xacro:if value="${camera_tower_size == 'small'}">
-      <xacro:pan_and_tilt>
-        <origin
-          rpy="0 0 0"
-          xyz="0.061228 0 0.402"/>
-      </xacro:pan_and_tilt>
-    </xacro:if> <!-- base_type == 'create3' && camera_tower_size == 'small' -->
-  </xacro:if> <!-- base_type == 'create3' -->
-  <!-- ********************************** Lidar **********************************  -->
-  <xacro:if value="$(arg use_lidar)">
+          xyz="-0.0345 0 0.010763"/>
+      </xacro:battery>
+    </xacro:if> <!-- base_type == 'create3' -->
+  </xacro:unless> <!-- !robot_model.startswith('locobotcmu_wx200') -->
+  <!-- ********************************** Camera Tower **********************************  -->
+  <xacro:if value="${robot_model_var.startswith('locobotcmu')}">
+    <xacro:locobotcmu_camera_tower/>
+  </xacro:if> <!-- robot_model.startswith('locobotcmu_wx200') -->
+  <xacro:unless value="${robot_model_var.startswith('locobotcmu')}">
     <xacro:if value="${base_type == 'kobuki'}">
       <xacro:if value="${camera_tower_size == 'large'}">
-        <xacro:lidar>
-          <origin
-            rpy="0 0 0"
-            xyz="-0.074 0 0.44425"/>
-        </xacro:lidar>
+        <xacro:camera_tower>
+          <origin
+            rpy="0 0 0"
+            xyz="-0.023997 -0.000044 0.08823"/>
+          <inertial>
+            <origin
+              rpy="0 0 0"
+              xyz="-0.0372211000 -0.0026114300 0.1744600000"/>
+            <mass value="2.366224"/>
+            <inertia
+              ixx="0.0628500000"
+              ixy="0.0002152000"
+              ixz="0.0065630000"
+              iyy="0.0546000000"
+              iyz="-0.0004738000"
+              izz="0.0179300000"/>
+          </inertial>
+        </xacro:camera_tower>
       </xacro:if> <!-- base_type == 'kobuki' && camera_tower_size == 'large' -->
       <xacro:if value="${camera_tower_size == 'small'}">
-        <xacro:lidar>
-          <origin
-            rpy="0 0 0"
-            xyz="-0.074 0 0.38425"/>
-        </xacro:lidar>
+        <xacro:camera_tower>
+          <origin
+            rpy="0 0 0"
+            xyz="-0.023997 -0.000044 0.08823"/>
+          <inertial>
+            <origin
+              rpy="0 0 0"
+              xyz="-0.0357703000 -0.0027068600 0.1560470000"/>
+            <mass value="2.282808"/>
+            <inertia
+              ixx="0.0461600000"
+              ixy="0.0002062000"
+              ixz="0.0052560000"
+              iyy="0.0384200000"
+              iyz="-0.0003600000"
+              izz="0.0169600000"/>
+          </inertial>
+        </xacro:camera_tower>
       </xacro:if> <!-- base_type == 'kobuki' && camera_tower_size == 'small' -->
     </xacro:if> <!-- base_type == 'kobuki' -->
     <xacro:if value="${base_type == 'create3'}">
       <xacro:if value="${camera_tower_size == 'large'}">
-        <xacro:lidar>
-          <origin
-            rpy="0 0 0"
-            xyz="-0.066095 0 0.462"/>
-        </xacro:lidar>
+        <xacro:camera_tower>
+          <origin
+            rpy="0 0 0"
+            xyz="-0.048271 0 0.10087"/>
+          <inertial>
+            <origin
+              rpy="0 0 0"
+              xyz="-0.025958 -0.003319 0.205872"/>
+            <mass value="2.514064"/>
+            <inertia
+              ixx="7.61E-02"
+              ixy="1.47E-04"
+              ixz="7.04E-03"
+              iyy="6.71E-02"
+              iyz="-9.41E-04"
+              izz="1.95E-02"/>
+          </inertial>
+        </xacro:camera_tower>
       </xacro:if> <!-- base_type == 'create3' && camera_tower_size == 'large' -->
       <xacro:if value="${camera_tower_size == 'small'}">
-        <xacro:lidar>
-          <origin
-            rpy="0 0 0"
-            xyz="-0.066095 0 0.402"/>
-        </xacro:lidar>
+        <xacro:camera_tower>
+          <origin
+            rpy="0 0 0"
+            xyz="-0.048271 0 0.10087"/>
+          <inertial>
+            <origin
+              rpy="0 0 0"
+              xyz="-0.024689 -0.003432 0.185408"/>
+            <mass value="2.430647"/>
+            <inertia
+              ixx="5.63E-02"
+              ixy="1.37E-04"
+              ixz="5.75E-03"
+              iyy="4.78E-02"
+              iyz="-7.70E-04"
+              izz="1.86E-02"/>
+          </inertial>
+        </xacro:camera_tower>
       </xacro:if> <!-- base_type == 'create3' && camera_tower_size == 'small' -->
     </xacro:if> <!-- base_type == 'create3' -->
-  </xacro:if> <!-- use_lidar -->
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