Commit message: modified urdf to launch locobotcmu, passed gazebo sim launch

File: interbotix_ros_xslocobots/interbotix_xslocobot_descriptions/urdf/pan_and_tilt.urdf.xacro (robot description, xacro)
@@ -9,5 +9,10 @@
         upper="${pi/2}"
         velocity="${pi}"/>
-      <xacro:insert_block name="origin"/>
+      <xacro:if value="${robot_model_var.startswith('locobotcmu')}">
+        <origin rpy="0 0 0" xyz="0.0240154841629213 -0.000373468229198185 0.4065"/>
+      </xacro:if> <!-- robot_model.startswith('locobotcmu_wx200') -->
+      <xacro:unless value="${robot_model_var.startswith('locobotcmu')}">
+        <xacro:insert_block name="origin"/>
+      </xacro:unless> <!-- !robot_model.startswith('locobotcmu_wx200') -->
       <parent
         link="${robot_name}/camera_tower_link"/>
@@ -19,38 +24,62 @@
     </joint>
     <link name="${robot_name}/pan_link">
-      <visual>
-        <origin
-          rpy="0 0 ${pi/2}"
-          xyz="0 0 0"/>
-        <geometry>
-          <mesh
-            filename="package://interbotix_xslocobot_descriptions/meshes/locobot_meshes/locobot_pan.stl"
-            scale="0.001 0.001 0.001"/>
-        </geometry>
-        <material name="interbotix_black"/>
-      </visual>
-      <collision>
-        <origin
-          rpy="0 0 ${pi/2}"
-          xyz="0 0 0"/>
-        <geometry>
-          <mesh
-            filename="package://interbotix_xslocobot_descriptions/meshes/locobot_meshes/locobot_pan.stl"
-            scale="0.001 0.001 0.001"/>
-        </geometry>
-      </collision>
-      <inertial>
-        <origin
-          rpy="0 0 ${pi/2}"
-          xyz="0.012 0.000496 0.018504"/>
-        <mass value="0.098997"/>
-        <inertia
-          ixx="0.0000276300"
-          ixy="0.0000000418"
-          ixz="0.0000005145"
-          iyy="0.0000204300"
-          iyz="-0.0000000421"
-          izz="0.0000276300"/>
-      </inertial>
+      <xacro:if value="${robot_model_var.startswith('locobotcmu')}">
+        <inertial>
+            <origin rpy="0 0 0" xyz="-1.35308431126191E-16 -2.97071395261028E-17 0.0220876265081744"/>
+            <mass value="0.0182769203076134"/>
+            <inertia ixx="1.32243845065555E-05" ixy="5.07660179129181E-13" ixz="1.067515220067E-20" iyy="7.13386116649085E-06" iyz="-1.32882457845217E-20" izz="7.83291781352837E-06"/>
+        </inertial>
+        <visual>
+            <origin rpy="0 0 0" xyz="0 0 0"/>
+            <geometry>
+                <mesh filename="package://interbotix_xslocobot_descriptions/meshes/cmu_locobot_meshes/tilt_link.STL"/>
+            </geometry>
+            <material name="">
+                <color rgba="0.250980392156863 0.250980392156863 0.250980392156863 1"/>
+            </material>
+        </visual>
+        <collision>
+            <origin rpy="0 0 0" xyz="0 0 0"/>
+            <geometry>
+                <mesh filename="package://interbotix_xslocobot_descriptions/meshes/cmu_locobot_meshes/tilt_link.STL"/>
+            </geometry>
+        </collision>
+      </xacro:if> <!-- robot_model.startswith('locobotcmu_wx200') -->
+      <xacro:unless value="${robot_model_var.startswith('locobotcmu')}">
+        <visual>
+          <origin
+            rpy="0 0 ${pi/2}"
+            xyz="0 0 0"/>
+          <geometry>
+            <mesh
+              filename="package://interbotix_xslocobot_descriptions/meshes/locobot_meshes/locobot_pan.stl"
+              scale="0.001 0.001 0.001"/>
+          </geometry>
+          <material name="interbotix_black"/>
+        </visual>
+        <collision>
+          <origin
+            rpy="0 0 ${pi/2}"
+            xyz="0 0 0"/>
+          <geometry>
+            <mesh
+              filename="package://interbotix_xslocobot_descriptions/meshes/locobot_meshes/locobot_pan.stl"
+              scale="0.001 0.001 0.001"/>
+          </geometry>
+        </collision>
+        <inertial>
+          <origin
+            rpy="0 0 ${pi/2}"
+            xyz="0.012 0.000496 0.018504"/>
+          <mass value="0.098997"/>
+          <inertia
+            ixx="0.0000276300"
+            ixy="0.0000000418"
+            ixz="0.0000005145"
+            iyy="0.0000204300"
+            iyz="-0.0000000421"
+            izz="0.0000276300"/>
+        </inertial>
+      </xacro:unless> <!-- !robot_model.startswith('locobotcmu_wx200') -->
     </link>
     <gazebo reference="${robot_name}/pan_link">
@@ -65,7 +94,12 @@
         upper="${radians(75)}"
         velocity="${pi}"/>
-      <origin
-        rpy="0 0 0"
-        xyz="0.025034 0 0.019"/>
+      <xacro:if value="${robot_model_var.startswith('locobotcmu')}">
+        <origin rpy="0 0 0" xyz="0 0 0.05"/>
+      </xacro:if> <!-- robot_model.startswith('locobotcmu_wx200') -->
+      <xacro:unless value="${robot_model_var.startswith('locobotcmu')}">
+        <origin
+          rpy="0 0 0"
+          xyz="0.025034 0 0.019"/>
+      </xacro:unless> <!-- !robot_model.startswith('locobotcmu_wx200') -->
       <parent
         link="${robot_name}/pan_link"/>
@@ -98,38 +132,62 @@
     </xacro:if>
     <link name="${robot_name}/tilt_link">
-      <visual>
-        <origin
-          rpy="0 0 ${pi/2}"
-          xyz="0 0 0"/>
-        <geometry>
-          <mesh
-            filename="package://interbotix_xslocobot_descriptions/meshes/locobot_meshes/locobot_tilt.stl"
-            scale="0.001 0.001 0.001"/>
-        </geometry>
-        <material name="interbotix_black"/>
-      </visual>
-      <collision>
-        <origin
-          rpy="0 0 ${pi/2}"
-          xyz="0 0 0"/>
-        <geometry>
-          <mesh
-            filename="package://interbotix_xslocobot_descriptions/meshes/locobot_meshes/locobot_tilt.stl"
-            scale="0.001 0.001 0.001"/>
-        </geometry>
-      </collision>
-      <inertial>
-        <origin
-          rpy="0 0 ${pi/2}"
-          xyz="0.0237737000 -0.0000016331 0.0000077432"/>
-        <mass value="0.019845"/>
-        <inertia
-          ixx="0.0000021677"
-          ixy="0.0000000000"
-          ixz="0.0000000001"
-          iyy="0.0000063634"
-          iyz="0.0000000003"
-          izz="0.0000066157"/>
-      </inertial>
+      <xacro:if value="${robot_model_var.startswith('locobotcmu')}">
+        <inertial>
+            <origin rpy="0 0 0" xyz="0.0168744200088311 -0.000442984145897884 -0.00405256422002387"/>
+            <mass value="0.0547677687275323"/>
+            <inertia ixx="1.07071738005716E-05" ixy="-1.46854788384565E-07" ixz="5.59529059364376E-08" iyy="1.77011620295824E-05" iyz="1.27587154712834E-09" izz="2.01583693170578E-05"/>
+        </inertial>
+        <visual>
+            <origin rpy="0 0 0" xyz="0 0 0"/>
+            <geometry>
+                <mesh filename="package://interbotix_xslocobot_descriptions/meshes/cmu_locobot_meshes/roll_link.STL"/>
+            </geometry>
+            <material name="">
+                <color rgba="0.792156862745098 0.819607843137255 0.933333333333333 1"/>
+            </material>
+        </visual>
+        <collision>
+            <origin rpy="0 0 0" xyz="0 0 0"/>
+            <geometry>
+                <mesh filename="package://interbotix_xslocobot_descriptions/meshes/cmu_locobot_meshes/roll_link.STL"/>
+            </geometry>
+        </collision>
+      </xacro:if> <!-- robot_model.startswith('locobotcmu_wx200') -->
+      <xacro:unless value="${robot_model_var.startswith('locobotcmu')}">
+        <visual>
+          <origin
+            rpy="0 0 ${pi/2}"
+            xyz="0 0 0"/>
+          <geometry>
+            <mesh
+              filename="package://interbotix_xslocobot_descriptions/meshes/locobot_meshes/locobot_tilt.stl"
+              scale="0.001 0.001 0.001"/>
+          </geometry>
+          <material name="interbotix_black"/>
+        </visual>
+        <collision>
+          <origin
+            rpy="0 0 ${pi/2}"
+            xyz="0 0 0"/>
+          <geometry>
+            <mesh
+              filename="package://interbotix_xslocobot_descriptions/meshes/locobot_meshes/locobot_tilt.stl"
+              scale="0.001 0.001 0.001"/>
+          </geometry>
+        </collision>
+        <inertial>
+          <origin
+            rpy="0 0 ${pi/2}"
+            xyz="0.0237737000 -0.0000016331 0.0000077432"/>
+          <mass value="0.019845"/>
+          <inertia
+            ixx="0.0000021677"
+            ixy="0.0000000000"
+            ixz="0.0000000001"
+            iyy="0.0000063634"
+            iyz="0.0000000003"
+            izz="0.0000066157"/>
+        </inertial>
+      </xacro:unless> <!-- !robot_model.startswith('locobotcmu_wx200') -->
     </link>
     <gazebo reference="${robot_name}/tilt_link">
@@ -138,7 +196,12 @@
     </gazebo>
     <joint name="camera" type="fixed">
-      <origin
-        rpy="0 0 0"
-        xyz="0.05318 0.0175 0.000009"/>
+      <xacro:if value="${robot_model_var.startswith('locobotcmu')}">
+        <origin rpy="0 0 0" xyz="0.06705 0 -0.00425"/>
+      </xacro:if> <!-- robot_model.startswith('locobotcmu_wx200') -->
+      <xacro:unless value="${robot_model_var.startswith('locobotcmu')}">
+        <origin
+          rpy="0 0 0"
+          xyz="0.05318 0.0175 0.000009"/>
+      </xacro:unless> <!-- !robot_model.startswith('locobotcmu_wx200') -->
       <parent
         link="${robot_name}/tilt_link"/>
@@ -150,41 +213,65 @@
     </gazebo>
     <link name="camera_${robot_name}_link">
-      <visual>
-        <origin
-          rpy="0 0 0"
-          xyz="0 0 0"/>
-        <geometry>
-          <mesh
-            filename="package://interbotix_xslocobot_descriptions/meshes/locobot_meshes/locobot_camera.stl"
-            scale="0.001 0.001 0.001"/>
-        </geometry>
-        <material name="">
-          <color
-            rgba="0.55 0.55 0.55 1"/>
-        </material>
-      </visual>
-      <collision>
-        <origin
-          rpy="0 0 0"
-          xyz="0 0 0"/>
-        <geometry>
-          <mesh
-            filename="package://interbotix_xslocobot_descriptions/meshes/locobot_meshes/locobot_camera.stl"
-            scale="0.001 0.001 0.001"/>
-        </geometry>
-      </collision>
-      <inertial>
-        <origin
-          rpy="0 0 0"
-          xyz="-0.008972 -0.015818 0.000003"/>
-        <mass value="0.072"/>
-        <inertia
-          ixx="0.0000465400"
-          ixy="0.0000003028"
-          ixz="0.0000000245"
-          iyy="0.0000069128"
-          iyz="0.0000000248"
-          izz="0.0000468600"/>
-      </inertial>
+      <xacro:if value="${robot_model_var.startswith('locobotcmu')}">
+        <inertial>
+            <origin rpy="0 0 0" xyz="-0.0132722976093535 0.00168171470080143 2.49829664994428E-06"/>
+            <mass value="0.0381925651163644"/>
+            <inertia ixx="2.4688255642946E-05" ixy="1.60697655569215E-07" ixz="1.2993241737711E-08" iyy="3.66669176935806E-06" iyz="1.30215657011203E-08" izz="2.48602467766615E-05"/>
+        </inertial>
+        <visual>
+            <origin rpy="0 0 0" xyz="0 0 0"/>
+            <geometry>
+                <mesh filename="package://interbotix_xslocobot_descriptions/meshes/cmu_locobot_meshes/camera_link.STL"/>
+            </geometry>
+            <material name="">
+                <color rgba="0.792156862745098 0.819607843137255 0.933333333333333 1"/>
+            </material>
+        </visual>
+        <collision>
+            <origin rpy="0 0 0" xyz="0 0 0"/>
+            <geometry>
+                <mesh filename="package://interbotix_xslocobot_descriptions/meshes/cmu_locobot_meshes/camera_link.STL"/>
+            </geometry>
+        </collision>
+      </xacro:if> <!-- robot_model.startswith('locobotcmu_wx200') -->
+      <xacro:unless value="${robot_model_var.startswith('locobotcmu')}">
+        <visual>
+          <origin
+            rpy="0 0 0"
+            xyz="0 0 0"/>
+          <geometry>
+            <mesh
+              filename="package://interbotix_xslocobot_descriptions/meshes/locobot_meshes/locobot_camera.stl"
+              scale="0.001 0.001 0.001"/>
+          </geometry>
+          <material name="">
+            <color
+              rgba="0.55 0.55 0.55 1"/>
+          </material>
+        </visual>
+        <collision>
+          <origin
+            rpy="0 0 0"
+            xyz="0 0 0"/>
+          <geometry>
+            <mesh
+              filename="package://interbotix_xslocobot_descriptions/meshes/locobot_meshes/locobot_camera.stl"
+              scale="0.001 0.001 0.001"/>
+          </geometry>
+        </collision>
+        <inertial>
+          <origin
+            rpy="0 0 0"
+            xyz="-0.008972 -0.015818 0.000003"/>
+          <mass value="0.072"/>
+          <inertia
+            ixx="0.0000465400"
+            ixy="0.0000003028"
+            ixz="0.0000000245"
+            iyy="0.0000069128"
+            iyz="0.0000000248"
+            izz="0.0000468600"/>
+        </inertial>
+      </xacro:unless> <!-- !robot_model.startswith('locobotcmu_wx200') -->
     </link>
     <gazebo reference="camera_${robot_name}_link">

File: interbotix_ros_xslocobots/interbotix_xslocobot_descriptions/urdf/plate.urdf.xacro (robot description, xacro)
@@ -40,3 +40,75 @@
     </gazebo>
   </xacro:macro>
+  <xacro:macro name="locobotcmu_plate">
+    <!-- plate 0, joint named as plate to be consistent with above -->
+    <joint name="plate" type="fixed">
+        <origin rpy="0 0 0" xyz="0.0973 0 0.0902375"/>
+        <parent link="${robot_name}/base_link"/>
+        <child link="${robot_name}/plate0_link"/>
+        <!-- <axis xyz="0 0 0"/> -->
+    </joint>
+    <link name="${robot_name}/plate0_link">
+        <inertial>
+            <origin rpy="0 0 0" xyz="0 0 0"/>
+            <mass value="0.640128902693298"/>
+            <inertia ixx="0.0212697824374231" ixy="-1.84819421839641E-07" ixz="0.00177278831625861" iyy="0.0200161122874848" iyz="1.82514218153984E-07" izz="0.00538401325307411"/>
+        </inertial>
+        <visual>
+            <origin rpy="0 0 0" xyz="0 0 0"/>
+            <geometry>
+                <mesh filename="package://interbotix_xslocobot_descriptions/meshes/cmu_locobot_meshes/plate.STL"/>
+            </geometry>
+            <material name="">
+                <color rgba="0.792156862745098 0.819607843137255 0.933333333333333 1"/>
+            </material>
+        </visual>
+        <collision>
+            <origin rpy="0 0 0" xyz="0 0 0"/>
+            <geometry>
+                <mesh filename="package://interbotix_xslocobot_descriptions/meshes/cmu_locobot_meshes/plate.STL"/>
+            </geometry>
+        </collision>
+    </link>
+    <!-- plate1, named as plate_link to be consistent with above -->
+    <joint name="${robot_name}/plate1_joint" type="fixed">
+        <origin rpy="0 0 0" xyz="0 0 0.0047625"/>
+        <parent link="${robot_name}/plate0_link"/>
+        <child link="${robot_name}/plate_link"/>
+        <axis xyz="0 0 0"/>
+    </joint>
+    <link name="${robot_name}/plate_link">
+        <inertial>
+            <origin rpy="0 0 0" xyz="0 0 0"/>
+            <mass value="0.640128902693298"/>
+            <inertia ixx="0.0212697824374231" ixy="-1.84819421839641E-07" ixz="0.00177278831625861" iyy="0.0200161122874848" iyz="1.82514218153984E-07" izz="0.00538401325307411"/>
+        </inertial>
+        <visual>
+            <origin rpy="0 0 0" xyz="0 0 0"/>
+            <geometry>
+                <mesh filename="package://interbotix_xslocobot_descriptions/meshes/cmu_locobot_meshes/plate.STL"/>
+            </geometry>
+            <material name="">
+                <color rgba="0.792156862745098 0.819607843137255 0.933333333333333 1"/>
+            </material>
+        </visual>
+        <collision>
+            <origin rpy="0 0 0" xyz="0 0 0"/>
+            <geometry>
+                <mesh filename="package://interbotix_xslocobot_descriptions/meshes/cmu_locobot_meshes/plate.STL"/>
+            </geometry>
+        </collision>
+    </link>
+    <gazebo reference="${robot_name}/plate0_link">
+      <material>Gazebo/DarkGrey</material>
+    </gazebo>
+    <gazebo reference="${robot_name}/plate_link">
+      <material>Gazebo/DarkGrey</material>
+    </gazebo>
+    <gazebo reference="plate">
+      <disableFixedJointLumping>true</disableFixedJointLumping>
+    </gazebo>
+    <gazebo reference="${robot_name}/plate1_joint">
+      <disableFixedJointLumping>true</disableFixedJointLumping>
+    </gazebo>
+  </xacro:macro>
 </robot>
