Commit message: update urdf for new cam

File: interbotix_ros_xslocobots/interbotix_xslocobot_descriptions/urdf/pan_and_tilt.urdf.xacro (robot description, xacro)
@@ -195,142 +195,151 @@
       <self_collide>true</self_collide>
     </gazebo>
-    <joint name="camera" type="fixed">
-      <xacro:if value="${robot_model_var.startswith('locobotcmu')}">
-        <origin rpy="0 0 0" xyz="0.06705 0 -0.00425"/>
-      </xacro:if> <!-- robot_model.startswith('locobotcmu_wx200') -->
-      <xacro:unless value="${robot_model_var.startswith('locobotcmu')}">
-        <origin
-          rpy="0 0 0"
-          xyz="0.05318 0.0175 0.000009"/>
-      </xacro:unless> <!-- !robot_model.startswith('locobotcmu_wx200') -->
-      <parent
-        link="${robot_name}/tilt_link"/>
-      <child
-        link="camera_${robot_name}_link"/>
-    </joint>
-    <gazebo reference="camera">
-      <disableFixedJointLumping>true</disableFixedJointLumping>
-    </gazebo>
-    <link name="camera_${robot_name}_link">
-      <xacro:if value="${robot_model_var.startswith('locobotcmu')}">
-        <inertial>
-            <origin rpy="0 0 0" xyz="-0.0132722976093535 0.00168171470080143 2.49829664994428E-06"/>
-            <mass value="0.0381925651163644"/>
-            <inertia ixx="2.4688255642946E-05" ixy="1.60697655569215E-07" ixz="1.2993241737711E-08" iyy="3.66669176935806E-06" iyz="1.30215657011203E-08" izz="2.48602467766615E-05"/>
-        </inertial>
-        <visual>
-            <origin rpy="0 0 0" xyz="0 0 0"/>
-            <geometry>
-                <mesh filename="package://interbotix_xslocobot_descriptions/meshes/cmu_locobot_meshes/camera_link.STL"/>
-            </geometry>
-            <material name="">
-                <color rgba="0.792156862745098 0.819607843137255 0.933333333333333 1"/>
-            </material>
-        </visual>
-        <collision>
-            <origin rpy="0 0 0" xyz="0 0 0"/>
-            <geometry>
-                <mesh filename="package://interbotix_xslocobot_descriptions/meshes/cmu_locobot_meshes/camera_link.STL"/>
-            </geometry>
-        </collision>
-      </xacro:if> <!-- robot_model.startswith('locobotcmu_wx200') -->
-      <xacro:unless value="${robot_model_var.startswith('locobotcmu')}">
-        <visual>
-          <origin
-            rpy="0 0 0"
-            xyz="0 0 0"/>
-          <geometry>
-            <mesh
-              filename="package://interbotix_xslocobot_descriptions/meshes/locobot_meshes/locobot_camera.stl"
-              scale="0.001 0.001 0.001"/>
-          </geometry>
-          <material name="">
-            <color
-              rgba="0.55 0.55 0.55 1"/>
-          </material>
-        </visual>
-        <collision>
-          <origin
-            rpy="0 0 0"
-            xyz="0 0 0"/>
-          <geometry>
-            <mesh
-              filename="package://interbotix_xslocobot_descriptions/meshes/locobot_meshes/locobot_camera.stl"
-              scale="0.001 0.001 0.001"/>
-          </geometry>
-        </collision>
-        <inertial>
-          <origin
-            rpy="0 0 0"
-            xyz="-0.008972 -0.015818 0.000003"/>
-          <mass value="0.072"/>
-          <inertia
-            ixx="0.0000465400"
-            ixy="0.0000003028"
-            ixz="0.0000000245"
-            iyy="0.0000069128"
-            iyz="0.0000000248"
-            izz="0.0000468600"/>
-        </inertial>
-      </xacro:unless> <!-- !robot_model.startswith('locobotcmu_wx200') -->
-    </link>
-    <gazebo reference="camera_${robot_name}_link">
-      <material>Gazebo/Grey</material>
-      <self_collide>true</self_collide>
-    </gazebo>
-    <!-- Adds a dummy link, libgazebo_ros_openni_kinect publishes from frame's z-axis -->
-    <!-- https://github.com/ros-simulation/gazebo_ros_pkgs/issues/243 -->
-    <joint name="camera_depth_joint" type="fixed">
-      <origin rpy="${-pi/2} 0 ${-pi/2}" xyz="0 0 0"/>
-      <parent link="camera_${robot_name}_link"/>
-      <child link="${robot_name}/camera_depth_link"/>
-    </joint>
-    <link name="${robot_name}/camera_depth_link">
-      <origin rpy="0 0 0" xyz="0 0 0"/>
-    </link>
-    <gazebo reference="camera_${robot_name}_link">
-      <sensor name="camera_frame_sensor" type="depth">
-        <always_on>true</always_on>
-        <update_rate>30.0</update_rate>
-        <camera>
-          <horizontal_fov>0.994837</horizontal_fov>
-          <image>
-            <format>R8G8B8</format>
-            <width>640</width>
-            <height>480</height>
-          </image>
-          <clip>
-            <near>0.01</near>
-            <far>10</far>
-          </clip>
-        </camera>
-        <plugin filename="libgazebo_ros_camera.so" name="camera_frame_controller">
-          <ros>
-            <namespace>/$(arg robot_name)</namespace>
-          </ros>
-          <alwaysOn>true</alwaysOn>
-          <updateRate>0.0</updateRate>
-          <cameraName>camera</cameraName>
-          <imageTopicName>color/image_raw</imageTopicName>
-          <cameraInfoTopicName>color/camera_info</cameraInfoTopicName>
-          <depthImageTopicName>aligned_depth_to_color/image_raw</depthImageTopicName>
-          <depthImageCameraInfoTopicName>aligned_depth_to_color/camera_info</depthImageCameraInfoTopicName>
-          <pointCloudTopicName>depth_registered/points</pointCloudTopicName>
-          <frameName>${robot_name}/camera_depth_link</frameName>
-          <pointCloudCutoff>0.01</pointCloudCutoff>
-          <pointCloudCutoffMax>10</pointCloudCutoffMax>
-          <distortionK1>0.00000001</distortionK1>
-          <distortionK2>0.00000001</distortionK2>
-          <distortionK3>0.00000001</distortionK3>
-          <distortionT1>0.00000001</distortionT1>
-          <distortionT2>0.00000001</distortionT2>
-          <CxPrime>0</CxPrime>
-          <Cx>0</Cx>
-          <Cy>0</Cy>
-          <focalLength>0</focalLength>
-          <hackBaseline>0</hackBaseline>
-        </plugin>
-      </sensor>
-    </gazebo>
+    <xacro:unless value="${robot_model_var.startswith('locobotcmu')}">
+        <joint name="camera" type="fixed">
+          <xacro:if value="${robot_model_var.startswith('locobotcmu')}">
+            <origin rpy="0 0 0" xyz="0.06705 0 -0.00425"/>
+          </xacro:if> <!-- robot_model.startswith('locobotcmu_wx200') -->
+          <xacro:unless value="${robot_model_var.startswith('locobotcmu')}">
+            <origin
+              rpy="0 0 0"
+              xyz="0.05318 0.0175 0.000009"/>
+          </xacro:unless> <!-- !robot_model.startswith('locobotcmu_wx200') -->
+          <parent
+            link="${robot_name}/tilt_link"/>
+          <child
+            link="camera_${robot_name}_link"/>
+        </joint>
+        <gazebo reference="camera">
+          <disableFixedJointLumping>true</disableFixedJointLumping>
+        </gazebo>
+        <link name="camera_${robot_name}_link">
+          <xacro:if value="${robot_model_var.startswith('locobotcmu')}">
+            <inertial>
+                <origin rpy="0 0 0" xyz="-0.0132722976093535 0.00168171470080143 2.49829664994428E-06"/>
+                <mass value="0.0381925651163644"/>
+                <inertia ixx="2.4688255642946E-05" ixy="1.60697655569215E-07" ixz="1.2993241737711E-08" iyy="3.66669176935806E-06" iyz="1.30215657011203E-08" izz="2.48602467766615E-05"/>
+            </inertial>
+            <visual>
+                <origin rpy="0 0 0" xyz="0 0 0"/>
+                <geometry>
+                    <mesh filename="package://interbotix_xslocobot_descriptions/meshes/cmu_locobot_meshes/camera_link.STL"/>
+                </geometry>
+                <material name="">
+                    <color rgba="0.792156862745098 0.819607843137255 0.933333333333333 1"/>
+                </material>
+            </visual>
+            <collision>
+                <origin rpy="0 0 0" xyz="0 0 0"/>
+                <geometry>
+                    <mesh filename="package://interbotix_xslocobot_descriptions/meshes/cmu_locobot_meshes/camera_link.STL"/>
+                </geometry>
+            </collision>
+          </xacro:if> <!-- robot_model.startswith('locobotcmu_wx200') -->
+          <xacro:unless value="${robot_model_var.startswith('locobotcmu')}">
+            <visual>
+              <origin
+                rpy="0 0 0"
+                xyz="0 0 0"/>
+              <geometry>
+                <mesh
+                  filename="package://interbotix_xslocobot_descriptions/meshes/locobot_meshes/locobot_camera.stl"
+                  scale="0.001 0.001 0.001"/>
+              </geometry>
+              <material name="">
+                <color
+                  rgba="0.55 0.55 0.55 1"/>
+              </material>
+            </visual>
+            <collision>
+              <origin
+                rpy="0 0 0"
+                xyz="0 0 0"/>
+              <geometry>
+                <mesh
+                  filename="package://interbotix_xslocobot_descriptions/meshes/locobot_meshes/locobot_camera.stl"
+                  scale="0.001 0.001 0.001"/>
+              </geometry>
+            </collision>
+            <inertial>
+              <origin
+                rpy="0 0 0"
+                xyz="-0.008972 -0.015818 0.000003"/>
+              <mass value="0.072"/>
+              <inertia
+                ixx="0.0000465400"
+                ixy="0.0000003028"
+                ixz="0.0000000245"
+                iyy="0.0000069128"
+                iyz="0.0000000248"
+                izz="0.0000468600"/>
+            </inertial>
+          </xacro:unless> <!-- !robot_model.startswith('locobotcmu_wx200') -->
+        </link>
+        <gazebo reference="camera_${robot_name}_link">
+          <material>Gazebo/Grey</material>
+          <self_collide>true</self_collide>
+        </gazebo>
+        <!-- Adds a dummy link, libgazebo_ros_openni_kinect publishes from frame's z-axis -->
+        <!-- https://github.com/ros-simulation/gazebo_ros_pkgs/issues/243 -->
+        <joint name="camera_depth_joint" type="fixed">
+          <origin rpy="${-pi/2} 0 ${-pi/2}" xyz="0 0 0"/>
+          <parent link="camera_${robot_name}_link"/>
+          <child link="${robot_name}/camera_depth_link"/>
+        </joint>
+        <link name="${robot_name}/camera_depth_link">
+          <origin rpy="0 0 0" xyz="0 0 0"/>
+        </link>
+        <gazebo reference="camera_${robot_name}_link">
+          <sensor name="camera_frame_sensor" type="depth">
+            <always_on>true</always_on>
+            <update_rate>30.0</update_rate>
+            <camera>
+              <horizontal_fov>0.994837</horizontal_fov>
+              <image>
+                <format>R8G8B8</format>
+                <width>640</width>
+                <height>480</height>
+              </image>
+              <clip>
+                <near>0.01</near>
+                <far>10</far>
+              </clip>
+            </camera>
+            <plugin filename="libgazebo_ros_camera.so" name="camera_frame_controller">
+              <ros>
+                <namespace>/$(arg robot_name)</namespace>
+              </ros>
+              <alwaysOn>true</alwaysOn>
+              <updateRate>0.0</updateRate>
+              <cameraName>camera</cameraName>
+              <imageTopicName>color/image_raw</imageTopicName>
+              <cameraInfoTopicName>color/camera_info</cameraInfoTopicName>
+              <depthImageTopicName>aligned_depth_to_color/image_raw</depthImageTopicName>
+              <depthImageCameraInfoTopicName>aligned_depth_to_color/camera_info</depthImageCameraInfoTopicName>
+              <pointCloudTopicName>depth_registered/points</pointCloudTopicName>
+              <frameName>${robot_name}/camera_depth_link</frameName>
+              <pointCloudCutoff>0.01</pointCloudCutoff>
+              <pointCloudCutoffMax>10</pointCloudCutoffMax>
+              <distortionK1>0.00000001</distortionK1>
+              <distortionK2>0.00000001</distortionK2>
+              <distortionK3>0.00000001</distortionK3>
+              <distortionT1>0.00000001</distortionT1>
+              <distortionT2>0.00000001</distortionT2>
+              <CxPrime>0</CxPrime>
+              <Cx>0</Cx>
+              <Cy>0</Cy>
+              <focalLength>0</focalLength>
+              <hackBaseline>0</hackBaseline>
+            </plugin>
+          </sensor>
+        </gazebo>
+    </xacro:unless> <!-- !robot_model.startswith('locobotcmu_wx200') -->
+    <xacro:if value="${robot_model_var.startswith('locobotcmu')}">
+      <xacro:arg name="use_nominal_extrinsics" default="false"/>
+      <xacro:include filename="$(find realsense2_description)/urdf/_d455.urdf.xacro" />
+      <xacro:sensor_d455 parent="${robot_name}/tilt_link" use_nominal_extrinsics="$(arg use_nominal_extrinsics)" name="camera_${robot_name}">
+        <origin xyz="0.052 0 -0.0145" rpy="0 0 0"/>
+      </xacro:sensor_d455>
+    </xacro:if> <!-- robot_model.startswith('locobotcmu_wx200') -->
   </xacro:macro>
 </robot>
